Commit message: 1. add webots simulation model of self developed robot 2. add joint effort limit for 6 joints

File: depalletizing_ws/src/robot_description/robots/robot_arm.urdf (robot description, URDF)
Before this commit: robot robot, 10 links, 9 joints
Joints:
- joint robot_joint1: limit lower=0.0 upper=2.15 effort=400 velocity=0.3 -> lower=0.0 upper=2.15 effort=1222 velocity=0.3
- joint robot_joint2: limit lower=-1.66 upper=1.66 effort=400 velocity=4.147 -> lower=-1.66 upper=1.66 effort=160 velocity=4.147
- joint robot_joint3: limit lower=-2.6 upper=2.6 effort=400 velocity=3.665 -> lower=-2.6 upper=2.6 effort=84 velocity=3.665
- joint robot_joint4: limit lower=-3.32 upper=3.32 effort=400 velocity=4.974 -> lower=-3.32 upper=3.32 effort=30 velocity=4.974
- joint robot_joint5: limit lower=-1.60 upper=1.85 effort=60 velocity=1.623 -> lower=-1.60 upper=1.85 effort=528 velocity=1.623
- joint robot_joint6: limit lower=-3.32 upper=3.32 effort=60 velocity=3.665 -> lower=-3.32 upper=3.32 effort=84 velocity=3.665

File: depalletizing_ws/src/robot_description/robots/robot_arm.xacro (robot description, xacro)
@@ -60,5 +60,5 @@
       <child link="${arm_id}_link1"/>
       <axis xyz="0 0 1"/>
-      <limit effort="400" lower="0.0" upper="2.15" velocity="0.3"/>
+      <limit effort="1222" lower="0.0" upper="2.15" velocity="0.3"/>
     </joint>
     <!-- link2 -->
@@ -87,5 +87,5 @@
       <child link="${arm_id}_link2"/>
       <axis xyz="0 0 1"/>
-      <limit effort="400" lower="-1.66" upper="1.66" velocity="4.147"/>
+      <limit effort="160" lower="-1.66" upper="1.66" velocity="4.147"/>
     </joint>
     <!-- link3 -->
@@ -115,5 +115,5 @@
       <child link="${arm_id}_link3"/>
       <axis xyz="0 0 1"/>
-      <limit effort="400" lower="-2.6" upper="2.6" velocity="3.665"/>
+      <limit effort="84" lower="-2.6" upper="2.6" velocity="3.665"/>
     </joint>
     <!-- link4 -->
@@ -144,5 +144,5 @@
       <child link="${arm_id}_link4"/>
       <axis xyz="0 0 1"/>
-      <limit effort="400" lower="-3.32" upper="3.32" velocity="4.974"/>
+      <limit effort="30" lower="-3.32" upper="3.32" velocity="4.974"/>
     </joint>
     <!-- link5 -->
@@ -173,5 +173,5 @@
       <child link="${arm_id}_link5"/>
       <axis xyz="0 0 1"/>
-      <limit effort="60" lower="-1.60" upper="1.85" velocity="1.623"/>
+      <limit effort="528" lower="-1.60" upper="1.85" velocity="1.623"/>
     </joint>
     <!-- link6 -->
@@ -184,5 +184,5 @@
       <child link="${arm_id}_link6"/>
       <axis xyz="0 0 1"/>
-      <limit effort="60" lower="-3.32" upper="3.32" velocity="3.665"/>
+      <limit effort="84" lower="-3.32" upper="3.32" velocity="3.665"/>
     </joint>
     <!-- gripper -->

Commit message: first version of depelletizing demo is completed

File: depalletizing_ws/src/robot_description/robots/robot_arm.urdf (robot description, URDF)
Before this commit: robot robot, 10 links, 9 joints
Joints:
- joint robot_joint2: limit lower=-1.66 upper=1.66 effort=160 velocity=4.147 -> lower=-1.9 upper=1.9 effort=160 velocity=4.147
- joint robot_joint4: limit lower=-3.32 upper=3.32 effort=30 velocity=4.974 -> lower=-2 upper=2 effort=30 velocity=4.974; origin xyz=0.500 0 -0.187 rpy=0 0 0 -> xyz=0.500 0 -0.187 rpy=0 0 1.5707963267948966
- joint robot_joint6: limit lower=-3.32 upper=3.32 effort=84 velocity=3.665 -> lower=-2 upper=2 effort=84 velocity=3.665; origin xyz=0.0 -0.120 0 rpy=1.5707963267948966 0 0 -> xyz=0.0 -0.120 0 rpy=1.5707963267948966 -1.5707963267948966 0

File: depalletizing_ws/src/robot_description/robots/robot_arm.xacro (robot description, xacro)
@@ -87,5 +87,5 @@
       <child link="${arm_id}_link2"/>
       <axis xyz="0 0 1"/>
-      <limit effort="160" lower="-1.66" upper="1.66" velocity="4.147"/>
+      <limit effort="160" lower="-1.9" upper="1.9" velocity="4.147"/>
     </joint>
     <!-- link3 -->
@@ -140,9 +140,9 @@
     <joint name="${arm_id}_joint4" type="revolute">
       <safety_controller k_position="100.0" k_velocity="40.0" soft_lower_limit="-3.32" soft_upper_limit="3.32"/>
-      <origin rpy="0 0 0" xyz="0.500 0 -0.187"/>
+      <origin rpy="0 0 ${pi/2}" xyz="0.500 0 -0.187"/>
       <parent link="${arm_id}_link3"/>
       <child link="${arm_id}_link4"/>
       <axis xyz="0 0 1"/>
-      <limit effort="30" lower="-3.32" upper="3.32" velocity="4.974"/>
+      <limit effort="30" lower="-2" upper="2" velocity="4.974"/>
     </joint>
     <!-- link5 -->
@@ -180,9 +180,9 @@
     <joint name="${arm_id}_joint6" type="revolute">
       <safety_controller k_position="100.0" k_velocity="40.0" soft_lower_limit="-3.32" soft_upper_limit="3.32"/>
-      <origin rpy="${pi/2} 0 0" xyz="0.0 -0.120 0"/>
+      <origin rpy="${pi/2} -${pi/2} 0" xyz="0.0 -0.120 0"/>
       <parent link="${arm_id}_link5"/>
       <child link="${arm_id}_link6"/>
       <axis xyz="0 0 1"/>
-      <limit effort="84" lower="-3.32" upper="3.32" velocity="3.665"/>
+      <limit effort="84" lower="-2" upper="2" velocity="3.665"/>
     </joint>
     <!-- gripper -->

Commit message: add a branch for ShenZhen field testing.

File: depalletizing_ws/src/robot_description/robots/robot_arm.urdf (robot description, URDF)
Before this commit: robot robot, 10 links, 9 joints
Joints:
- joint robot_joint1: limit lower=0.0 upper=2.15 effort=1222 velocity=0.3 -> lower=0.0 upper=2.15 effort=1222 velocity=0.2

Commit message: update new urdf model for new robot

File: depalletizing_ws/src/robot_description/robots/robot_arm.urdf (robot description, URDF)
Before this commit: robot robot, 10 links, 9 joints
Links:
- link robot_link6: mass None -> 2.0; geometry collision mesh filename=package://robot_description/meshes/collision/link6.stl; visual mesh filename=package://robot_description/meshes/visual/link6.dae
Joints:
- joint bottom_joint: origin xyz=0 0 0.075 rpy=0 0 0 -> xyz=0 0 0.070 rpy=0 0 0
- joint robot_joint1: origin xyz=0.157 0 0.324 rpy=0 0 0 -> xyz=0.157 0 0.48 rpy=0 0 0
- joint robot_joint3: origin xyz=0.500 0 0.1833 rpy=0 0 0 -> xyz=0.49999 -0.0036478 -0.1833 rpy=0 0 0
- joint robot_joint4: origin xyz=0.500 0 -0.187 rpy=0 0 1.5707963267948966 -> xyz=0.49997 -0.005232 -0.187 rpy=0 0 1.5707963267948966
- joint robot_joint5: axis 0 0 1 -> 0 -1 0; limit lower=-1.60 upper=1.85 effort=528 velocity=1.623 -> lower=-1.85 upper=1.85 effort=528 velocity=1.623; origin xyz=0 0 0 rpy=1.5707963267948966 0 0 -> xyz=-0.0013802 -0.13189 0 rpy=0 1.5707963267948966 0
- joint robot_joint6: axis 0 0 1 -> -1 0 0; origin xyz=0.0 -0.120 0 rpy=1.5707963267948966 -1.5707963267948966 0 -> xyz=0.13687 0.13047 0 rpy=-1.5707963267948966 0 0
- joint robot_joint7: origin xyz=0.100 0.0 0.047 rpy=0 0 0 -> xyz=0.031498 0.0 0 rpy=0 1.5707963267948966 0
- joint tcp_joint: origin xyz=0 0 0.06887 rpy=0 0 0 -> xyz=0.1 0 0.06887 rpy=0 0 0

Commit message: update new 1st joint

File: depalletizing_ws/src/robot_description/robots/robot_arm.urdf (robot description, URDF)
Before this commit: robot robot, 10 links, 9 joints
Joints:
- joint robot_joint1: origin xyz=0.157 0 0.48 rpy=0 0 0 -> xyz=0.157 0 0.566 rpy=0 0 0
